File: SensorBoard_ver2.0.kicad_pcb (KiCad board)
At the start: 2 copper layers, 7 parts

Commit message: Add files via upload
Parts:
- added C1: ?, Capacitor_SMD:C_0603_1608Metric, F.Cu at (58.1, 55.1)
- added C10: 1μF, Capacitor_SMD:C_0603_1608Metric, F.Cu at (62.1, 60.1)
- added C11: C, Capacitor_SMD:C_0603_1608Metric, F.Cu at (62.1, 62.6)
- added C12: C, Capacitor_SMD:C_0603_1608Metric, F.Cu at (62.1, 65.1)
- added C13: 0.1μF, Capacitor_SMD:C_0603_1608Metric, F.Cu at (62.1, 67.6)
- added C2: ?, Capacitor_SMD:C_0603_1608Metric, F.Cu at (58.1, 57.6)
- added C3: 0.1μF, Capacitor_SMD:C_0603_1608Metric, F.Cu at (58.1, 60.1)
- added C4: 0.1μF, Capacitor_SMD:C_0603_1608Metric, F.Cu at (58.1, 62.6)
- added C5: ?, Capacitor_SMD:C_0603_1608Metric, F.Cu at (58.1, 65.1)
- added C6: ?, Capacitor_SMD:C_0603_1608Metric, F.Cu at (58.1, 67.6)
- added C7: 0.1μF, Capacitor_SMD:C_0603_1608Metric, F.Cu at (58.1, 70.1)
- added C8: 0.1μF, Capacitor_SMD:C_0603_1608Metric, F.Cu at (62.1, 55.1)
- added C9: 0.1μF, Capacitor_SMD:C_0603_1608Metric, F.Cu at (62.1, 57.6)
- added D1: LED, LED_SMD:LED_0603_1608Metric, F.Cu at (77.3, 12.9)
- added D2: LED, LED_SMD:LED_0603_1608Metric, F.Cu at (77.3, 15.5)
- added D3: LED, LED_SMD:LED_0603_1608Metric, F.Cu at (77.3, 18.1)
- added FB1: FerriteBead, Inductor_SMD:L_0603_1608Metric, F.Cu at (62.1, 70.1)
- added J1: CANConn, Connector_JST:JST_XA_S04B-XASK-1_1x04_P2.50mm_Horizontal, F.Cu at (177.8, 93.0)
- added J10: Limit3-B, Connector_JST:JST_XA_B02B-XASK-1_1x02_P2.50mm_Vertical, F.Cu at (97.0, 133.6)
- added J12: Limit2-A, Connector_JST:JST_XA_B02B-XASK-1_1x02_P2.50mm_Vertical, F.Cu at (97.0, 142.0)
- added J13: Limit2-B, Connector_JST:JST_XA_B02B-XASK-1_1x02_P2.50mm_Vertical, F.Cu at (106.6, 108.2)
- added J14: Limit4-A, Connector_JST:JST_XA_B02B-XASK-1_1x02_P2.50mm_Vertical, F.Cu at (106.6, 116.7)
- added J15: Limit4-B, Connector_JST:JST_XA_B02B-XASK-1_1x02_P2.50mm_Vertical, F.Cu at (106.6, 125.1)
- added J16: Abso, Connector_JST:JST_XA_S04B-XASK-1_1x04_P2.50mm_Horizontal, F.Cu at (205.8, 93.0)
- added J17: Abso, Connector_JST:JST_XA_S04B-XASK-1_1x04_P2.50mm_Horizontal, F.Cu at (219.8, 93.0)
- added J18: STLink, Connector_PinHeader_1.27mm:PinHeader_2x07_P1.27mm_Vertical_SMD, F.Cu at (72.3, 76.9)
- added J19: Abso, Connector_JST:JST_XA_S04B-XASK-1_1x04_P2.50mm_Horizontal, F.Cu at (235.2, 90.8)
- added J2: CANConn, Connector_JST:JST_XA_S04B-XASK-1_1x04_P2.50mm_Horizontal, F.Cu at (191.8, 93.0)
- added J20: VCP, Connector_JST:JST_XA_S04B-XASK-1_1x04_P2.50mm_Horizontal, F.Cu at (109.7, 69.5)
- added J21: Abso, Connector_JST:JST_XA_S04B-XASK-1_1x04_P2.50mm_Horizontal, F.Cu at (235.2, 76.8)
- added J22: Abso, Connector_JST:JST_XA_S04B-XASK-1_1x04_P2.50mm_Horizontal, F.Cu at (235.2, 62.8)
- added J3: Enc1, Connector_JST:JST_XA_S04B-XASK-1_1x04_P2.50mm_Horizontal, F.Cu at (227.0, 57.8)
- added J4: Enc2, Connector_JST:JST_XA_S04B-XASK-1_1x04_P2.50mm_Horizontal, F.Cu at (213.0, 57.8)
- added J5: Enc3, Connector_JST:JST_XA_S04B-XASK-1_1x04_P2.50mm_Horizontal, F.Cu at (199.0, 57.8)
- added J6: Enc4, Connector_JST:JST_XA_S04B-XASK-1_1x04_P2.50mm_Horizontal, F.Cu at (185.0, 57.8)
- added J7: Limit1-A, Connector_JST:JST_XA_B02B-XASK-1_1x02_P2.50mm_Vertical, F.Cu at (97.0, 108.2)
- added J8: Limit1-B, Connector_JST:JST_XA_B02B-XASK-1_1x02_P2.50mm_Vertical, F.Cu at (97.0, 116.7)
- added J9: Limit3-A, Connector_JST:JST_XA_B02B-XASK-1_1x02_P2.50mm_Vertical, F.Cu at (97.0, 125.1)
- added JP1: VCC⇔5V Short, Jumper:SolderJumper-2_P1.3mm_Open_RoundedPad1.0x1.5mm, F.Cu at (33.0, 80.3)
- added R1: 10kΩ, Resistor_SMD:R_0603_1608Metric, F.Cu at (66.2, 55.1)
- added R2: 10kΩ, Resistor_SMD:R_0603_1608Metric, F.Cu at (66.2, 57.6)
- added R3: 10kΩ, Resistor_SMD:R_0603_1608Metric, F.Cu at (66.2, 60.1)
- added R4: 10kΩ, Resistor_SMD:R_0603_1608Metric, F.Cu at (66.2, 62.6)
- added R6: 120Ω, Resistor_SMD:R_0603_1608Metric, F.Cu at (66.2, 65.1)
- added R7: 10kΩ, Resistor_SMD:R_0603_1608Metric, F.Cu at (66.2, 67.6)
- added R8: 120Ω, Resistor_SMD:R_0603_1608Metric, F.Cu at (66.2, 70.1)
- added SW1: CAN_Terminal, Connector_PinHeader_2.54mm:PinHeader_1x03_P2.54mm_Vertical, F.Cu at (193.0, 32.3)
- added SW2: IDSetSW, Connector_PinHeader_2.54mm:PinHeader_1x03_P2.54mm_Vertical, F.Cu at (197.0, 32.3)
- added SW3: Enc⇔Lim Change, Connector_PinHeader_2.54mm:PinHeader_1x03_P2.54mm_Vertical, F.Cu at (201.0, 32.3)
- added SW5: RS485_Terminal, Connector_PinHeader_2.54mm:PinHeader_1x03_P2.54mm_Vertical, F.Cu at (161.6, 112.3)
- added U1: L7805, Package_TO_SOT_SMD:TO-252-2, F.Cu at (47.6, 74.3)
- added U2: ATA6561, Package_SO:SOIC-8_3.9x4.9mm_P1.27mm, F.Cu at (72.4, 57.2)
- added U3: 3.3V Regulator, Package_TO_SOT_SMD:SOT-223, F.Cu at (45.2, 75.0)
- added U4: STM32F303K8Tx, Package_QFP:LQFP-32_7x7mm_P0.8mm, F.Cu at (192.5, 82.5)
- added U5: MAX3485, Package_SO:SOIC-8_3.9x4.9mm_P1.27mm, F.Cu at (72.4, 63.8)
- added Y1: Crystal, Crystal:Crystal_SMD_HC49-SD, F.Cu at (48.0, 81.7)

Commit message: 回路図の更新・PCBを作成
そんなもん
Parts:
- removed the J13 at (106.6, 108.2)
- removed the J14 at (106.6, 116.7)
- removed the J15 at (106.6, 125.1)
- added J11: Limit4, Connector_JST:JST_XA_S02B-XASK-1_1x02_P2.50mm_Horizontal, F.Cu at (108.8, 38.6)
- added J20: Enc5, Connector_JST:JST_XA_S04B-XASK-1_1x04_P2.50mm_Horizontal, F.Cu at (220.2, 93.5)
- added JP2: FB-Short, Jumper:SolderJumper-2_P1.3mm_Open_TrianglePad1.0x1.5mm, B.Cu at (141.5, 49.5)
- J10: value Limit3-B -> USB_C; footprint Connector_JST:JST_XA_B02B-XASK-1_1x02_P2.50mm_Vertical -> MyUSB_C:PowerOnlyUSB_C
- J12: value Limit2-A -> Limit3; footprint Connector_JST:JST_XA_B02B-XASK-1_1x02_P2.50mm_Vertical -> Connector_JST:JST_XA_S02B-XASK-1_1x02_P2.50mm_Horizontal
- J17: renamed from J20; footprint Connector_JST:JST_XA_S04B-XASK-1_1x04_P2.50mm_Horizontal -> Connector_JST:JST_XA_B04B-XASK-1_1x04_P2.50mm_Vertical
- J7: value Limit1-A -> LimitConn; footprint Connector_JST:JST_XA_B02B-XASK-1_1x02_P2.50mm_Vertical -> Connector_JST:JST_XA_S05B-XASK-1_1x05_P2.50mm_Horizontal
- J8: value Limit1-B -> Limit1; footprint Connector_JST:JST_XA_B02B-XASK-1_1x02_P2.50mm_Vertical -> Connector_JST:JST_XA_S02B-XASK-1_1x02_P2.50mm_Horizontal
- J9: value Limit3-A -> Limit2; footprint Connector_JST:JST_XA_B02B-XASK-1_1x02_P2.50mm_Vertical -> Connector_JST:JST_XA_S02B-XASK-1_1x02_P2.50mm_Horizontal
- JP1: footprint Jumper:SolderJumper-2_P1.3mm_Open_RoundedPad1.0x1.5mm -> Jumper:SolderJumper-2_P1.3mm_Open_TrianglePad1.0x1.5mm
- moved C6 169.4 mm to (227.0, 81.5)
- moved U3 167.7 mm to (212.7, 83.2), turned to 0 degrees
- moved Y1 165.6 mm to (213.0, 67.5), turned to 90 degrees
- moved U1 153.9 mm to (201.2, 83.2), turned to 180 degrees
- moved C5 153.9 mm to (210.3, 88.0)
- moved C1 151.0 mm to (205.5, 88.0), turned to 180 degrees
- moved C2 148.8 mm to (205.5, 78.5), turned to 180 degrees
- moved U2 114.5 mm to (186.0, 71.3), turned to 180 degrees
- moved R6 113.9 mm to (180.0, 63.5), turned to -90 degrees
- moved U5 113.6 mm to (186.0, 63.5), turned to 180 degrees
- moved J12 105.6 mm to (118.3, 38.6)
- moved SW3 104.8 mm to (285.5, 94.2)
- moved SW2 104.0 mm to (280.5, 94.2)
- moved SW1 103.2 mm to (275.5, 94.2)
- moved J9 86.5 mm to (99.2, 38.6)
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- renumbered J16 to J13, J17 to J14, J18 to J15, J19 to J16, J21 to J18, J22 to J19
Connections:
- J10 pad 1: /EncB_3 -> +5V
- J12 pad 1: /EncA_2 -> /Limit3
- J7 pad 1: /EncA_1 -> /Limit1
- J7 pad 2: GND -> /Limit2
- J8 pad 1: /EncB_1 -> /Limit1
- J9 pad 1: /EncA_3 -> /Limit2
- U4 pad 29: /LED1 -> /EncA_5
- U4 pad 30: /LED2 -> /EncB_5
- U4 pad 9: /LimitMode -> unconnected-(U4-PA3-Pad9)
Routing:
- net VCC: track 0.00 -> 29.1 mm
- net +5V: track 0.00 -> 4.87 mm, vias 0 -> 3
- net /RS485_A: track 0.00 -> 3.63 mm
- net /RS485_B: track 0.00 -> 3.63 mm
- net +3.3VA: track 0.00 -> 0.10 mm, vias 0 -> 1
- net +3.3V: track 0.00 -> 0.09 mm, vias 0 -> 2
- net GND: vias 0 -> 36
- added copper zone on B.Cu, net GND
- added copper zone on F.Cu, net GND

Commit message: 基板作成
締まらない、なんか違う
Parts:
- removed J10: USB_C, MyUSB_C:PowerOnlyUSB_C
- removed SW3: Enc⇔Lim Change, Connector_PinHeader_2.54mm:PinHeader_1x03_P2.54mm_Vertical
- JP2: moved to F.Cu
- moved D1 204.1 mm to (272.1, 73.7)
- moved D2 204.1 mm to (272.1, 76.3)
- moved D3 204.1 mm to (272.1, 78.9)
- moved C10 197.5 mm to (258.0, 34.5)
- moved C11 197.5 mm to (258.0, 37.0)
- moved C12 197.5 mm to (258.0, 39.5)
- moved C13 197.5 mm to (258.0, 42.0)
- moved C8 197.5 mm to (258.0, 29.5)
- moved C9 197.5 mm to (258.0, 32.0)
- moved C3 197.5 mm to (254.0, 34.5)
- moved C4 197.5 mm to (254.0, 37.0)
- moved C7 197.5 mm to (254.0, 44.5)
- moved R1 197.5 mm to (262.0, 29.5)
- moved R2 197.5 mm to (262.0, 32.0)
- moved R3 197.5 mm to (262.0, 34.5)
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Connections:
- U3 pad 4: (no net) -> +3.3V
- U4 pad 27: /AbsoSW -> /EncA_1
- U4 pad 28: /IDSet -> /EncB_1
- U4 pad 6: /EncA_1 -> /AbsoSW
- U4 pad 7: /EncB_1 -> /IDSet
- U4 pad 9: unconnected-(U4-PA3-Pad9) -> /LED
Routing:
- net VCC: track 29.1 -> 0.00 mm
- net +5V: track 4.87 -> 0.00 mm, vias 3 -> 0
- net /CTRL: track 0.00 -> 1.27 mm
- net /RS485_A: track 3.63 -> 2.60 mm
- net /RS485_B: track 3.63 -> 2.60 mm
- net +3.3VA: track 0.10 -> 0.00 mm, vias 1 -> 0
- net +3.3V: track 0.09 -> 0.00 mm, vias 2 -> 0

Commit message: だいたい完成
だいたい完成しました
あとはタイプシーやらシルクやらを決めるだけ
Parts:
- removed ? (x3): , 
- removed J11: Limit4, Connector_JST:JST_XA_S02B-XASK-1_1x02_P2.50mm_Horizontal
- removed J12: Limit3, Connector_JST:JST_XA_S02B-XASK-1_1x02_P2.50mm_Horizontal
- removed J17: VCP, Connector_JST:JST_XA_B04B-XASK-1_1x04_P2.50mm_Vertical
- removed J7: LimitConn, Connector_JST:JST_XA_S05B-XASK-1_1x05_P2.50mm_Horizontal
- removed J8: Limit1, Connector_JST:JST_XA_S02B-XASK-1_1x02_P2.50mm_Horizontal
- removed J9: Limit2, Connector_JST:JST_XA_S02B-XASK-1_1x02_P2.50mm_Horizontal
- removed SW5: RS485_Terminal, Connector_PinHeader_2.54mm:PinHeader_1x03_P2.54mm_Vertical
- added R5: 120Ω, Resistor_SMD:R_0603_1608Metric, F.Cu at (61.6, 111.6)
- moved R2 227.9 mm to (39.2, 79.9)
- moved R3 227.9 mm to (39.2, 82.4)
- moved SW1 224.4 mm to (58.3, 114.6), turned to 90 degrees
- moved D1 212.8 mm to (59.4, 80.4)
- moved R1 204.4 mm to (64.0, 80.4), turned to 180 degrees
- moved U1 194.1 mm to (78.6, 91.0)
- moved C2 190.7 mm to (74.4, 96.2)
- moved R4 188.4 mm to (86.5, 105.5)
- moved C1 188.2 mm to (74.4, 85.8)
- moved JP1 183.6 mm to (70.8, 91.1), turned to -90 degrees
- moved C4 174.4 mm to (90.8, 98.5)
- moved R8 171.4 mm to (103.5, 109.8), turned to 180 degrees
- moved C3 170.5 mm to (95.9, 98.4)
- moved C8 166.4 mm to (102.6, 89.0), turned to 180 degrees
- moved R7 165.6 mm to (110.5, 109.0)
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Connections:
- C5 pad 1: VCC -> +5V
- R8 pad 1: /RS485_A -> /RS485_B
- R8 pad 2: Net-(SW5-A) -> /RS485_A
- U3 pad 3: VCC -> +5V
Routing:
- net +5V: track 0.00 -> 217.0 mm, vias 0 -> 10
- net +3.3V: track 0.00 -> 136.7 mm, vias 0 -> 11
- net /RS485_A: track 2.60 -> 78.4 mm, vias 0 -> 1
- net /RS485_B: track 2.60 -> 77.8 mm, vias 0 -> 1
- net /CANH: track 0.00 -> 55.6 mm, vias 0 -> 1
- net /CANL: track 0.00 -> 49.0 mm
- net /EncB_4: track 0.00 -> 42.7 mm
- net /VCPRX: track 0.00 -> 42.3 mm, vias 0 -> 2
- net /SWDIO: track 0.00 -> 41.6 mm, vias 0 -> 2
- net /EncA_1: track 0.00 -> 41.4 mm
- net /EncA_4: track 0.00 -> 41.1 mm
- net /EncB_1: track 0.00 -> 39.8 mm
- net VCC: track 0.00 -> 39.7 mm
- net /SWCLK: track 0.00 -> 39.0 mm, vias 0 -> 2
- net /VCPTX: track 0.00 -> 34.7 mm, vias 0 -> 2
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Other:
- board outline added: 93 x 56.2 mm
- board text added: "${REFERENCE}"
- board text added: "CAN Power ↓ LED"

Commit message: 多分最終稿
色々修正等
Parts:
- removed C13: 0.1μF, Capacitor_SMD:C_0603_1608Metric
- removed JP2: FB-Short, Jumper:SolderJumper-2_P1.3mm_Open_TrianglePad1.0x1.5mm
- added C14: 0.1μF, Capacitor_SMD:C_0603_1608Metric, F.Cu at (93.7, 89.0)
- added D4: LED, LED_SMD:LED_0603_1608Metric, F.Cu at (136.0, 94.9)
- added H5: Hamada, MySilcscreen:Hamada, B.Cu at (134.0, 92.8)
- added J10: USB_C, MyUSB_C:PowerOnlyUSB_C, F.Cu at (141.9, 91.5)
- added R9: 10kΩ, Resistor_SMD:R_0603_1608Metric, F.Cu at (133.0, 94.9)
- added SW3: Reset, MySW:SMD_MySW1, F.Cu at (145.2, 114.0)
- added SW4: IDSetSW, Connector_PinHeader_2.54mm:PinHeader_1x03_P2.54mm_Vertical, F.Cu at (142.2, 108.8)
- added SW5: Terminal, Connector_PinHeader_2.54mm:PinHeader_1x03_P2.54mm_Vertical, F.Cu at (86.5, 98.8)
- C1, C2: value ? -> 10μF; footprint Capacitor_SMD:C_0603_1608Metric -> Capacitor_SMD:C_0805_2012Metric
- C11, C12: value C -> 33pF?
- moved R2 104.0 mm to (143.2, 78.0)
- moved R3 104.0 mm to (143.2, 81.4)
- moved D3 97.0 mm to (147.2, 81.4), turned to 180 degrees
- moved D2 97.0 mm to (147.2, 78.0), turned to 180 degrees
- moved C7 61.9 mm to (115.4, 106.8), turned to 180 degrees
- moved C10 61.8 mm to (115.4, 102.7), turned to 180 degrees
- moved C9 37.0 mm to (137.3, 113.9), turned to 90 degrees
- moved SW2 33.0 mm to (143.8, 98.9), turned to 0 degrees
- moved R6 14.5 mm to (85.0, 95.8), turned to 0 degrees
- moved J15 5.71 mm to (130.7, 103.6)
- moved R8 4.85 mm to (108.2, 108.8), turned to 90 degrees
- moved U5 3.43 mm to (92.6, 92.9), turned to 180 degrees
- moved R7 3.30 mm to (110.4, 105.7)
- moved H3 1.60 mm to (60.4, 70.6)
- moved H4 1.40 mm to (145.5, 70.6)
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Connections:
- J20 pad 2: /EncA_5 -> /EncA_1
- J20 pad 3: /EncB_5 -> /EncB_1
- J3 pad 2: /EncA_1 -> /EncA_0
- J3 pad 3: /EncB_1 -> /EncB_0
- R6 pad 1: /RS485_A -> Net-(SW5-B)
- U4 pad 27: /EncA_1 -> /EncA_0
- U4 pad 28: /EncB_1 -> /EncB_0
- U4 pad 29: /EncA_5 -> /EncA_1
- U4 pad 30: /EncB_5 -> /EncB_1
- U4 pad 6: /AbsoSW -> /EncSW
Routing:
- net /RS485_A: track 78.4 -> 175.7 mm, vias 1 -> 3
- net /RS485_B: track 77.8 -> 170.0 mm, vias 1 -> 2
- net /EncSW: track 0.00 -> 43.5 mm, vias 0 -> 2
- net /EncA_0: track 0.00 -> 41.2 mm
- net /EncB_0: track 0.00 -> 39.6 mm
- net /IDSet: track 0.00 -> 38.0 mm, vias 0 -> 2
- net +5V: track 217.0 -> 246.6 mm
- net /EncA_5: track 29.1 -> 0.00 mm
- net /EncB_5: track 27.5 -> 0.00 mm
- net /LED: track 0.00 -> 26.4 mm, vias 0 -> 2
- net /NRST: track 32.0 -> 53.9 mm, vias 2 -> 3
- net /EncB_1: track 39.8 -> 27.4 mm
- net /EncA_1: track 41.4 -> 28.9 mm
- net /VCPTX: track 34.7 -> 28.4 mm
- net /VCPRX: track 42.3 -> 37.1 mm
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Other:
- board size 93 x 56.2 mm -> 93.1 x 58 mm
- board text added: "+3.3V"
- board text added: "+5V"
- board text added: "CAN"
- board text added: "CAN Power"
- board text added: "Designed by Hama"
- board text added: "Enc SW"
- board text added: "Enc0"
- board text added: "Enc1"
- board text added: "Enc2"
- board text added: "Enc3"
- board text added: "Enc4"
- board text added: "Firmware:Jaga"
- board text added: "IDSet Base⇔+4"
- board text added: "LED"
- board text added: "ON"
- board text added: "Power Only"
- board text added: "RS485 TerminalSW"
- board text added: "RS485:0"
- board text added: "RS485:1"
- board text added: "RS485:2"
- board text added: "RS485:3"
- board text added: "RS485:4"
- board text added: "Reset SW"
- board text added: "STLink"
- board text added: "SensorBoard Ver 1.0"
- board text added: "↙CAN TerminalSW"
- board text removed: "${REFERENCE}"
- board text removed: "CAN Power ↓ LED"

Commit message: 大改造する前のバックアップ
大改造して、失敗したときのバックアップです
Parts:
- removed U3: 3.3V Regulator, Package_TO_SOT_SMD:SOT-223
- added IC1: MIC5504-3.3YM5-T5, SOT95P280X130-5N:SOT95P280X130-5N, F.Cu at (131.4, 85.0)
- added R10: 10kΩ, Resistor_SMD:R_0603_1608Metric, F.Cu at (126.7, 83.8)
- C5, C6: value ? -> 1μF
- moved C6 0.90 mm to (135.9, 86.2)
- moved C5 0.81 mm to (136.0, 83.8)
Connections:
- SW3 pad 2: /NRST -> GND
Routing:
- net +3.3V: track 136.6 -> 121.9 mm, vias 12 -> 15
- net GND: track 0.00 -> 14.0 mm, vias 114 -> 119
- net +5V: track 246.6 -> 252.6 mm, vias 10 -> 11
- net /RS485_A: track 175.7 -> 171.3 mm
- net /RS485_B: track 170.0 -> 165.8 mm
- net Net-(IC1-EN): track 0.00 -> 2.99 mm

Commit message: 大改造したあと　ver01
特になし、アップロードしたファイル間違えてるかもしれないくらい？
Parts:
- removed FB1: FerriteBead, Inductor_SMD:L_0603_1608Metric
- removed H5: Hamada, MySilcscreen:Hamada
- removed J10: USB_C, MyUSB_C:PowerOnlyUSB_C
- removed SW5: Terminal, Connector_PinHeader_2.54mm:PinHeader_1x03_P2.54mm_Vertical
- moved H4 84.7 mm to (67.0, 102.2)
- moved H3 78.2 mm to (131.9, 102.2)
- moved C6 59.5 mm to (87.5, 120.7), turned to 180 degrees
- moved D2 58.0 mm to (135.4, 134.8)
- moved R2 57.9 mm to (131.9, 134.8)
- moved D3 57.3 mm to (135.4, 137.5)
- moved R3 57.2 mm to (131.9, 137.5)
- moved C5 56.7 mm to (87.4, 113.0), turned to 180 degrees
- moved IC1 55.0 mm to (87.2, 117.7)
- moved R10 50.0 mm to (87.4, 114.7), turned to 180 degrees
- moved J15 44.8 mm to (93.2, 128.2), turned to 0 degrees
- moved J16 39.9 mm to (130.7, 116.7), turned to 90 degrees
- moved C8 39.1 mm to (107.8, 127.7)
- moved SW2 38.8 mm to (116.8, 126.7), turned to -90 degrees
- moved J1 38.2 mm to (68.5, 123.9)
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Connections:
- R6 pad 1: Net-(SW5-B) -> /RS485_B
- R6 pad 2: /RS485_B -> /RS485_A
- SW3 pad 1: /NRST -> GND
- SW3 pad 2: GND -> /NRST
- U4 pad 5: +3.3VA -> +3.3V
Routing:
- net /RS485_A: track 171.3 -> 113.9 mm, vias 3 -> 2
- net /RS485_B: track 165.8 -> 113.5 mm
- net +5V: track 252.6 -> 214.3 mm, vias 11 -> 6
- net /SWDIO: track 36.4 -> 5.80 mm, vias 2 -> 0
- net /SWCLK: track 33.9 -> 5.99 mm, vias 2 -> 0
- net /EncSW: track 43.5 -> 16.2 mm, vias 2 -> 1
- net /NRST: track 53.9 -> 27.3 mm, vias 3 -> 2
- net /IDSet: track 38.0 -> 12.4 mm, vias 2 -> 1
- net +3.3V: track 121.9 -> 97.6 mm, vias 15 -> 8
- net /VCPRX: track 37.1 -> 14.2 mm
- net /LED: track 26.4 -> 6.71 mm, vias 2 -> 0
- net /CANH: track 55.4 -> 37.6 mm
- net /CANL: track 48.8 -> 33.9 mm
- net /EncA_4: track 41.5 -> 27.2 mm
- net /EncB_4: track 43.1 -> 28.9 mm
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Other:
- board size 93.1 x 58 mm -> 82.5 x 50 mm
- board text added: "Abso_0"
- board text added: "Abso_1"
- board text added: "Abso_2"
- board text added: "Abso_3"
- board text added: "Abso_4"
- board text added: "EncSW"
- board text added: "Enc_0"
- board text added: "Enc_1"
- board text added: "Enc_2"
- board text added: "Enc_3"
- board text added: "Enc_4"
- board text added: "IDSet"
- board text removed: "+3.3V"
- board text removed: "+5V"
- board text removed: "CAN Power"
- board text removed: "Designed by Hama"
- board text removed: "Enc SW"
- board text removed: "Enc0"
- board text removed: "Enc1"
- board text removed: "Enc2"
- board text removed: "Enc3"
- board text removed: "Enc4"
- board text removed: "Firmware:Jaga"
- board text removed: "IDSet Base⇔+4"
- board text removed: "LED"
- board text removed: "ON"
- board text removed: "Power Only"
- board text removed: "RS485 TerminalSW"
- board text removed: "RS485:0"
- board text removed: "RS485:1"
- board text removed: "RS485:2"
- board text removed: "RS485:3"
- board text removed: "RS485:4"
- board text removed: "Reset SW"
- board text removed: "STLink"
- board text removed: "SensorBoard Ver 1.0"
- board text removed: "↙CAN TerminalSW"
